File: v_2/KiCad/midi-v2-circuit.kicad_pcb (KiCad board)
At the start: 2 copper layers, 33 parts, among them CON1 AVR-ISP-10, CON2 AVR-ISP-10, CON3 AVR-ISP-10, J1 Screw_Terminal_01x10, J2 Conn_01x04, J3 DIN-8, J4 Conn_01x17, J5 Conn_01x04, J6 USB_B, J7 to_midi_adapter_USB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

Commit message: ready for atmega 90 deg rotate branch
Routing:
- net +5V: track 340.0 -> 357.7 mm
- net midi-raw-signal-power: track 129.3 -> 133.4 mm
Changed lines of the file:
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@@
 (kicad_pcb (version 4) (host pcbnew 4.0.7-e2-6376~58~ubuntu16.04.1)
   (general
-    (links 128)
+    (links 0)
     (no_connects 19)
     (area 0 0 0 0)
     (thickness 1.6)
     (drawings 0)
-    (tracks 645)
+    (tracks 651)
     (zones 0)
     (modules 33)
@@
     (pad_drill 0.762)
     (pad_to_mask_clearance 0.2)
-    (aux_axis_origin 0 0)
+    (aux_axis_origin 260.985 30.734)
     (visible_elements FFFFFF7F)
     (pcbplotparams
@@
     (add_net "Net-(J6-Pad2)")
     (add_net "Net-(J6-Pad3)")
-    (add_net "Net-(J8-Pad1)")
-    (add_net "Net-(J8-Pad3)")
     (add_net "Net-(RV1-PadB1A)")
     (add_net "Net-(RV1-PadB1B)")
@@
   (segment (start 204.368 70.365) (end 202.837 68.834) (width 0.2) (layer F.Cu) (net 4))
   (segment (start 202.837 68.834) (end 202.712 68.834) (width 0.2) (layer F.Cu) (net 4))
+  (segment (start 165.3375 164.4015) (end 165.4375 164.4015) (width 0.25) (layer F.Cu) (net 5))
+  (segment (start 173.0375 151.087) (end 173.0375 149.987) (width 0.25) (layer F.Cu) (net 5))
+  (segment (start 166.898999 157.225501) (end 173.0375 151.087) (width 0.25) (layer F.Cu) (net 5))
+  (segment (start 166.898999 162.940001) (end 166.898999 157.225501) (width 0.25) (layer F.Cu) (net 5))
+  (segment (start 165.4375 164.4015) (end 166.898999 162.940001) (width 0.25) (layer F.Cu) (net 5))
   (segment (start 173.101 144.653) (end 197.993 144.653) (width 0.25) (layer B.Cu) (net 5))
   (segment (start 197.993 144.653) (end 208.788 133.858) (width 0.25) (layer B.Cu) (net 5))
@@
   (segment (start 223.708001 101.750001) (end 208.368 86.41) (width 0.25) (layer F.Cu) (net 44))
   (segment (start 208.368 86.41) (end 208.368 85.36) (width 0.25) (layer F.Cu) (net 44))
-  (segment (start 189.738 128.016) (end 189.738 126.916) (width 0.25) (layer F.Cu) (net 49))
   (segment (start 199.318 84.04) (end 199.318 83.51) (width 0.25) (layer F.Cu) (net 49))
   (segment (start 199.318 117.336) (end 199.318 84.04) (width 0.25) (layer F.Cu) (net 49))
+  (segment (start 189.738 128.016) (end 189.738 126.916) (width 0.25) (layer F.Cu) (net 49))
   (segment (start 189.738 126.916) (end 199.318 117.336) (width 0.25) (layer F.Cu) (net 49))
   (segment (start 167.132 150.067) (end 159.94 150.067) (width 0.25) (layer F.Cu) (net 50))
@@
   (segment (start 178.1175 149.987) (end 178.967499 149.137001) (width 0.25) (layer F.Cu) (net 54))
   (segment (start 178.967499 149.137001) (end 178.967499 138.962499) (width 0.25) (layer F.Cu) (net 54))
+  (segment (start 168.0375 164.4015) (end 172.1485 164.4015) (width 0.25) (layer F.Cu) (net 55))
   (segment (start 170.942 101.346) (end 176.956601 95.331399) (width 0.25) (layer B.Cu) (net 55))
   (segment (start 176.956601 95.331399) (end 176.956601 78.931471) (width 0.25) (layer B.Cu) (net 55))
