File: v_2/KiCad/_autosave-midi-v2-circuit.kicad_pcb (KiCad board)
At the start: 2 copper layers, 36 parts, among them CON1 IDC-14, CON2 AVR-ISP-10, CON3 IDC-14, J1 Screw_Terminal_01x14, J2 Conn_01x04, J3 DIN-8, J4 Conn_01x17, J6 USB_B, J7 to_midi_adapter_USB, J8 to_midi_adapter_MIDI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

Commit message: rotation done, design stable enough for merging
Parts:
- added REF**: MountingHole_3mm, Mounting_Holes:MountingHole_3mm, F.Cu at (119.4, 73.7)
- added REF**: MountingHole_3mm, Mounting_Holes:MountingHole_3mm, F.Cu at (78.7, 73.7)
- added REF**: MountingHole_3mm, Mounting_Holes:MountingHole_3mm, F.Cu at (119.4, 114.3)
- added REF**: MountingHole_3mm, Mounting_Holes:MountingHole_3mm, F.Cu at (78.7, 114.3)
- J1: value Screw_Terminal_01x14 -> Screw_Terminal_01x12; footprint Pin_Headers:Pin_Header_Straight_1x14_Pitch2.54mm -> TerminalBlocks_Phoenix:TerminalBlock_Phoenix_MPT-2.54mm_12pol
- moved RV1 6.56 mm to (99.1, 94.0)
- moved J1 2.57 mm to (86.5, 111.3), turned to 0 degrees
- moved C10 1.63 mm to (105.4, 81.6)
- moved C11 1.63 mm to (105.4, 75.8)
- moved C8 1.63 mm to (109.7, 75.8)
- moved C9 1.63 mm to (109.7, 81.7)
- moved CON1 1.63 mm to (116.0, 97.5)
Connections:
- CON1 pad 10: button-3 -> button-4
- CON1 pad 12: button-4 -> button-2
- CON1 pad 9: button-2 -> button-3
- CON3 pad 1: knob-pot-4 -> joystick-pot-2
- CON3 pad 10: button-3 -> button-4
- CON3 pad 12: button-4 -> button-2
- CON3 pad 2: slide-pot-1 -> joystick-pot-1
- CON3 pad 3: knob-pot-3 -> knob-pot-4
- CON3 pad 4: slide-pot-2 -> knob-pot-3
- CON3 pad 6: joystick-pot-1 -> knob-pot-1
- CON3 pad 7: knob-pot-1 -> slide-pot-2
- CON3 pad 8: joystick-pot-2 -> slide-pot-1
- CON3 pad 9: button-2 -> button-3
- J1 pad 10: knob-pot-4 -> button-2
- J1 pad 11: button-1 -> button-3
- J1 pad 12: button-2 -> button-4
- J1 pad 3: joystick-pot-1 -> slide-pot-1
- J1 pad 4: joystick-pot-2 -> slide-pot-2
- J1 pad 5: slide-pot-1 -> knob-pot-1
- J1 pad 6: slide-pot-2 -> knob-pot-2
- J1 pad 7: knob-pot-1 -> knob-pot-3
- J1 pad 8: knob-pot-2 -> knob-pot-4
- J1 pad 9: knob-pot-3 -> button-1
Routing:
- net button-1: track 33.1 -> 92.9 mm
- net button-4: track 41.6 -> 94.7 mm
- net slide-pot-1: track 41.5 -> 84.1 mm
- net slide-pot-2: track 42.6 -> 82.5 mm
- net knob-pot-1: track 45.2 -> 82.0 mm
- net knob-pot-2: track 45.2 -> 79.4 mm
- net knob-pot-3: track 47.3 -> 78.4 mm
- net knob-pot-4: track 51.1 -> 79.0 mm
- net button-2: track 32.0 -> 55.7 mm
- net +5V: track 460.3 -> 481.7 mm
- net joystick-pot-1: track 106.0 -> 95.8 mm
- net joystick-pot-2: track 93.0 -> 86.2 mm
- net GND: track 416.7 -> 410.2 mm
- net button-3: track 36.4 -> 34.9 mm
- added copper zone on B.Cu, net GND

Commit message: autosave file update
Routing:
- net +5V: track 481.7 -> 424.2 mm
- net button-2: track 55.7 -> 96.6 mm
- net button-3: track 34.9 -> 74.2 mm
- net button-4: track 94.7 -> 79.9 mm
- net button-1: track 92.9 -> 82.3 mm
