File: v_2/KiCad/midi-v2-circuit.sch (KiCad schematic (older format))
At the start: 33 parts, among them CON1 AVR-ISP-10, CON2 AVR-ISP-10, CON3 AVR-ISP-10, J1 Screw_Terminal_01x10, J2 Conn_01x04, J3 DIN-8, J4 Conn_01x17, J5 Conn_01x04, J6 USB_B, J7 to_midi_adapter_USB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

Commit message: rotation done, design stable enough for merging
Parts:
- removed CON1: AVR-ISP-10, Connectors_IDC:IDC-Header_2x05_Pitch2.54mm_Angled, symbol AVR-ISP-10
- removed CON3: AVR-ISP-10, Connectors_IDC:IDC-Header_2x05_Pitch2.54mm_Straight, symbol AVR-ISP-10
- removed J1: Screw_Terminal_01x10, TerminalBlocks_Phoenix:TerminalBlock_Phoenix_MPT-2.54mm_10pol, symbol Screw_Terminal_01x10
- removed J5: Conn_01x04, Pin_Headers:Pin_Header_Straight_1x04_Pitch2.54mm, symbol Conn_01x04
- added C10, C11, C8, C9: 100n, Capacitors_SMD:C_0805_HandSoldering, symbol C
- added CON1: IDC-14, Connectors_IDC:IDC-Header_2x07_Pitch2.54mm_Angled, symbol IDC-14
- added CON3: IDC-14, Connectors_IDC:IDC-Header_2x07_Pitch2.54mm_Straight, symbol IDC-14
- added J1: Screw_Terminal_01x12, TerminalBlocks_Phoenix:TerminalBlock_Phoenix_MPT-2.54mm_12pol, symbol Screw_Terminal_01x12
- R2, R3: value 3.7k -> 4.7k
Connections:
- wire segments 108 -> 127

Commit message: adc first success
Parts:
- added R10, R11, R12, R13, R6, R7: 330, Resistors_SMD:R_0805_HandSoldering, symbol R
Connections:
- wire segments 127 -> 135
Changed lines of the file:
@@
 L GND #PWR026
 U 1 1 5B2DB672
-P 1150 4725
-F 0 "#PWR026" H 1150 4475 50  0001 C CNN
-F 1 "GND" H 1150 4575 50  0000 C CNN
-F 2 "" H 1150 4725 50  0001 C CNN
-F 3 "" H 1150 4725 50  0001 C CNN
-	1    1150 4725
-	1    0    0    -1
-$EndComp
-Text GLabel 2050 5025 0    60   Input ~ 0
+P 900 4450
+F 0 "#PWR026" H 900 4200 50  0001 C CNN
+F 1 "GND" H 900 4300 50  0000 C CNN
+F 2 "" H 900 4450 50  0001 C CNN
+F 3 "" H 900 4450 50  0001 C CNN
+	1    900  4450
+	1    0    0    -1
+$EndComp
+Text GLabel 1625 5125 0    60   Input ~ 0
 knob-pot-1
-Text GLabel 2050 5125 0    60   Input ~ 0
+Text GLabel 1625 5025 0    60   Input ~ 0
 knob-pot-2
-Text GLabel 2050 5225 0    60   Input ~ 0
+Text GLabel 1625 4925 0    60   Input ~ 0
 knob-pot-3
-Text GLabel 2050 5325 0    60   Input ~ 0
+Text GLabel 1625 4825 0    60   Input ~ 0
 knob-pot-4
-Text GLabel 2050 4825 0    60   Input ~ 0
+Text GLabel 1625 5325 0    60   Input ~ 0
 slide-pot-1
-Text GLabel 2050 4925 0    60   Input ~ 0
+Text GLabel 1625 5225 0    60   Input ~ 0
 slide-pot-2
 $Comp
@@
 	1150 4625 2050 4625
 Wire Wire Line
-	1150 4725 2050 4725
+	1025 4725 2050 4725
 Wire Notes Line
 	575  2525 575  7675
@@
 Wire Wire Line
 	2000 6850 2300 6850
+Text GLabel 2050 5625 0    60   Input ~ 0
+button-1
+Text GLabel 2050 5725 0    60   Input ~ 0
+button-2
 Text GLabel 2050 5425 0    60   Input ~ 0
-button-1
+button-3
 Text GLabel 2050 5525 0    60   Input ~ 0
-button-2
-Text GLabel 2050 5625 0    60   Input ~ 0
-button-3
-Text GLabel 2050 5725 0    60   Input ~ 0
 button-4
 $Comp
@@
 Text GLabel 10150 5700 2    60   Input ~ 0
 button-4
+$Comp
+L R R6
+U 1 1 5B34137C
+P 1900 5325
+F 0 "R6" V 1850 5150 50  0000 C CNN
+F 1 "330" V 1900 5325 50  0000 C CNN
+F 2 "Resistors_SMD:R_0805_HandSoldering" V 1830 5325 50  0001 C CNN
+F 3 "" H 1900 5325 50  0001 C CNN
+	1    1900 5325
+	0    1    1    0
+$EndComp
+Wire Wire Line
+	1025 4725 1025 4450
+Wire Wire Line
+	1025 4450 900  4450
+$Comp
+L R R7
+U 1 1 5B342758
+P 1900 5225
+F 0 "R7" V 1850 5050 50  0000 C CNN
+F 1 "330" V 1900 5225 50  0000 C CNN
+F 2 "Resistors_SMD:R_0805_HandSoldering" V 1830 5225 50  0001 C CNN
+F 3 "" H 1900 5225 50  0001 C CNN
+	1    1900 5225
+	0    1    1    0
+$EndComp
+$Comp
+L R R10
+U 1 1 5B342C8C
+P 1900 5125
+F 0 "R10" V 1850 4950 50  0000 C CNN
+F 1 "330" V 1900 5125 50  0000 C CNN
+F 2 "Resistors_SMD:R_0805_HandSoldering" V 1830 5125 50  0001 C CNN
+F 3 "" H 1900 5125 50  0001 C CNN
+	1    1900 5125
+	0    1    1    0
+$EndComp
+$Comp
+L R R11
+U 1 1 5B342C92
+P 1900 5025
+F 0 "R11" V 1850 4850 50  0000 C CNN
+F 1 "330" V 1900 5025 50  0000 C CNN
+F 2 "Resistors_SMD:R_0805_HandSoldering" V 1830 5025 50  0001 C CNN
+F 3 "" H 1900 5025 50  0001 C CNN
+	1    1900 5025
+	0    1    1    0
+$EndComp
+$Comp
+L R R12
+U 1 1 5B342D6E
+P 1900 4925
+F 0 "R12" V 1850 4750 50  0000 C CNN
+F 1 "330" V 1900 4925 50  0000 C CNN
+F 2 "Resistors_SMD:R_0805_HandSoldering" V 1830 4925 50  0001 C CNN
+F 3 "" H 1900 4925 50  0001 C CNN
+	1    1900 4925
+	0    1    1    0
+$EndComp
+$Comp
+L R R13
+U 1 1 5B342D74
+P 1900 4825
+F 0 "R13" V 1850 4650 50  0000 C CNN
+F 1 "330" V 1900 4825 50  0000 C CNN
+F 2 "Resistors_SMD:R_0805_HandSoldering" V 1830 4825 50  0001 C CNN
+F 3 "" H 1900 4825 50  0001 C CNN
+	1    1900 4825
+	0    1    1    0
+$EndComp
+Wire Wire Line
+	1750 5325 1625 5325
+Wire Wire Line
+	1625 5225 1750 5225
+Wire Wire Line
+	1750 5125 1625 5125
+Wire Wire Line
+	1625 5025 1750 5025
+Wire Wire Line
+	1750 4925 1625 4925
+Wire Wire Line
+	1625 4825 1750 4825
 $EndSCHEMATC

Commit message: improvements before first pcb order
Parts:
- added R14, R15, R16, R17: 10k, Resistors_SMD:R_0805_HandSoldering, symbol device:R
- C1, C10, C11, C2, C3, C4, C5, C6, C7, C8, C9: symbol C -> device:C
- CON1, CON3: symbol IDC-14 -> midi-v2-circuit-rescue:IDC-14
- CON2: symbol AVR-ISP-10 -> atmel:AVR-ISP-10
- D1, D2: symbol LED -> device:LED
- J1: symbol Screw_Terminal_01x12 -> conn:Screw_Terminal_01x12
- J2, J7: symbol Conn_01x04 -> conn:Conn_01x04
- J3: symbol DIN-8 -> conn:DIN-8
- J4: symbol Conn_01x17 -> conn:Conn_01x17
- J6: symbol USB_B -> conn:USB_B
- J8: symbol Conn_01x03 -> conn:Conn_01x03
- J9: symbol Conn_01x02 -> conn:Conn_01x02
- L1: footprint Inductors_SMD:L_1812_HandSoldering -> Inductors_SMD:L_0805_HandSoldering; symbol L -> device:L
- R1, R10, R11, R12, R13, R2, R3, R4, R5, R6, R7, R8, R9: symbol R -> device:R
- RV1: symbol Joystick-switch-POT_Dual -> midi-v2-circuit-rescue:Joystick-switch-POT_Dual
- SW2: symbol SW_Push -> switches:SW_Push
- U1: symbol ATMEGA32-16AU -> atmel:ATMEGA32-16AU
- Y1: symbol Crystal -> device:Crystal
Connections:
- wire segments 135 -> 172
Other:
- moved on the sheet: CON3

Commit message: prototyping ordered PCB, USART working, problem with keyboard keys
Parts:
- C1, C10, C11, C2, C3, C4, C5, C6, C7, C8, C9: symbol device:C -> midi-v2-circuit-rescue:C-device
- CON2: symbol atmel:AVR-ISP-10 -> midi-v2-circuit-rescue:AVR-ISP-10-atmel
- D1, D2: symbol device:LED -> midi-v2-circuit-rescue:LED-device
- J1: symbol conn:Screw_Terminal_01x12 -> midi-v2-circuit-rescue:Screw_Terminal_01x12-conn
- J2, J7: symbol conn:Conn_01x04 -> midi-v2-circuit-rescue:Conn_01x04-conn
- J3: symbol conn:DIN-8 -> midi-v2-circuit-rescue:DIN-8-conn
- J4: symbol conn:Conn_01x17 -> midi-v2-circuit-rescue:Conn_01x17-conn
- J6: symbol conn:USB_B -> midi-v2-circuit-rescue:USB_B-conn
- J8: symbol conn:Conn_01x03 -> midi-v2-circuit-rescue:Conn_01x03-conn
- J9: symbol conn:Conn_01x02 -> midi-v2-circuit-rescue:Conn_01x02-conn
- L1: symbol device:L -> midi-v2-circuit-rescue:L-device
- R1, R10, R11, R12, R13, R14, R15, R16, R17, R2, R3, R4, R5, R6, R7, R8, R9: symbol device:R -> midi-v2-circuit-rescue:R-device
- SW2: symbol switches:SW_Push -> midi-v2-circuit-rescue:SW_Push-switches
- U1: symbol atmel:ATMEGA32-16AU -> midi-v2-circuit-rescue:ATMEGA32-16AU-atmel
- Y1: symbol device:Crystal -> midi-v2-circuit-rescue:Crystal-device
Changed lines of the file:
@@
 $EndDescr
 $Comp
-L atmel:ATMEGA32-16AU U1
+L midi-v2-circuit-rescue:ATMEGA32-16AU-atmel U1
 U 1 1 5B2AD854
 P 5075 5275
@@
 button-4
 $Comp
-L conn:Conn_01x17 J4
+L midi-v2-circuit-rescue:Conn_01x17-conn J4
 U 1 1 5B2AEA28
 P 10400 3925
@@
 note-13
 $Comp
-L atmel:AVR-ISP-10 CON2
+L midi-v2-circuit-rescue:AVR-ISP-10-atmel CON2
 U 1 1 5B2AEEE8
 P 6175 1350
@@
 $EndComp
 $Comp
-L device:C C5
+L midi-v2-circuit-rescue:C-device C5
 U 1 1 5B2B8A3A
 P 5075 2875
@@
 $EndComp
 $Comp
-L device:C C6
+L midi-v2-circuit-rescue:C-device C6
 U 1 1 5B2B8C4B
 P 5525 2875
@@
 $EndComp
 $Comp
-L device:C C7
+L midi-v2-circuit-rescue:C-device C7
 U 1 1 5B2B8C9C
 P 5975 2875
@@
 $EndComp
 $Comp
-L device:C C4
+L midi-v2-circuit-rescue:C-device C4
 U 1 1 5B2B7A4D
 P 4625 2875
@@
 RST
 $Comp
-L switches:SW_Push SW2
+L midi-v2-circuit-rescue:SW_Push-switches SW2
 U 1 1 5B2B95B3
 P 3575 3575
@@
 $EndComp
 $Comp
-L device:R R1
+L midi-v2-circuit-rescue:R-device R1
 U 1 1 5B2B99E0
 P 3825 3425
@@
 $EndComp
 $Comp
-L device:Crystal Y1
+L midi-v2-circuit-rescue:Crystal-device Y1
 U 1 1 5B2BA77D
 P 3875 4175
@@
 $EndComp
 $Comp
-L device:C C1
+L midi-v2-circuit-rescue:C-device C1
 U 1 1 5B2BAED4
 P 3525 3975
@@
 $EndComp
 $Comp
-L device:C C2
+L midi-v2-circuit-rescue:C-device C2
 U 1 1 5B2BAF8F
 P 3525 4375
@@
 $EndComp
 $Comp
-L device:C C3
+L midi-v2-circuit-rescue:C-device C3
 U 1 1 5B2BBEE0
 P 3925 4775
@@
 $EndComp
 $Comp
-L device:L L1
+L midi-v2-circuit-rescue:L-device L1
 U 1 1 5B2BC3A2
 P 6275 2875
@@
 SCL
 $Comp
-L conn:Conn_01x04 J2
+L midi-v2-circuit-rescue:Conn_01x04-conn J2
 U 1 1 5B2C07E4
 P 7925 3200
@@
 $EndComp
 $Comp
-L device:R R2
+L midi-v2-circuit-rescue:R-device R2
 U 1 1 5B2C1345
 P 7375 2750
@@
 $EndComp
 $Comp
-L device:R R3
+L midi-v2-circuit-rescue:R-device R3
 U 1 1 5B2C1C9B
 P 7575 2750
@@
 $EndComp
 $Comp
-L device:R R4
+L midi-v2-circuit-rescue:R-device R4
 U 1 1 5B2D2B8E
 P 3575 1225
@@
 $EndComp
 $Comp
-L device:R R5
+L midi-v2-circuit-rescue:R-device R5
 U 1 1 5B2D55DF
 P 4975 1225
@@
 NoConn ~ 2275 3175
 $Comp
-L conn:DIN-8 J3
+L midi-v2-circuit-rescue:DIN-8-conn J3
 U 1 1 5B2EB01F
 P 4200 1325
@@
 NoConn ~ 4200 1625
 $Comp
-L conn:USB_B J6
+L midi-v2-circuit-rescue:USB_B-conn J6
 U 1 1 5B302844
 P 1325 1350
@@
 $EndComp
 $Comp
-L conn:Conn_01x04 J7
+L midi-v2-circuit-rescue:Conn_01x04-conn J7
 U 1 1 5B3041BE
 P 2375 1250
@@
 $EndComp
 $Comp
-L conn:Conn_01x03 J8
+L midi-v2-circuit-rescue:Conn_01x03-conn J8
 U 1 1 5B306C6E
 P 4675 2050
@@
 $EndComp
 $Comp
-L conn:Conn_01x02 J9
+L midi-v2-circuit-rescue:Conn_01x02-conn J9
 U 1 1 5B30BFB9
 P 7700 1300
@@
 $EndComp
 $Comp
-L device:LED D1
+L midi-v2-circuit-rescue:LED-device D1
 U 1 1 5B3116B9
 P 7375 1850
@@
 $EndComp
 $Comp
-L device:R R8
+L midi-v2-circuit-rescue:R-device R8
 U 1 1 5B312423
 P 7375 1550
@@
 $EndComp
 $Comp
-L device:LED D2
+L midi-v2-circuit-rescue:LED-device D2
 U 1 1 5B313961
 P 8450 1650
@@
 $EndComp
 $Comp
-L device:R R9
+L midi-v2-circuit-rescue:R-device R9
 U 1 1 5B313D52
 P 8450 1350
@@
 midi-raw-signal-data
 $Comp
-L device:C C8
+L midi-v2-circuit-rescue:C-device C8
 U 1 1 5B31F54F
 P 8275 5050
@@
 $EndComp
 $Comp
-L device:C C9
+L midi-v2-circuit-rescue:C-device C9
 U 1 1 5B31F7B1
 P 8275 5275
@@
 $EndComp
 $Comp
-L device:C C10
+L midi-v2-circuit-rescue:C-device C10
 U 1 1 5B31F842
 P 8275 5500
@@
 $EndComp
 $Comp
-L device:C C11
+L midi-v2-circuit-rescue:C-device C11
 U 1 1 5B31F8CC
 P 8275 5725
@@
 button-4
 $Comp
-L conn:Screw_Terminal_01x12 J1
+L midi-v2-circuit-rescue:Screw_Terminal_01x12-conn J1
 U 1 1 5B315AAE
 P 2250 5125
@@
 button-4
 $Comp
-L device:R R6
+L midi-v2-circuit-rescue:R-device R6
 U 1 1 5B34137C
 P 1900 5325
@@
 	1025 4450 900  4450
 $Comp
-L device:R R7
+L midi-v2-circuit-rescue:R-device R7
 U 1 1 5B342758
 P 1900 5225
@@
 $EndComp
 $Comp
-L device:R R10
+L midi-v2-circuit-rescue:R-device R10
 U 1 1 5B342C8C
 P 1900 5125
@@
 $EndComp
 $Comp
-L device:R R11
+L midi-v2-circuit-rescue:R-device R11
 U 1 1 5B342C92
 P 1900 5025
@@
 $EndComp
 $Comp
-L device:R R12
+L midi-v2-circuit-rescue:R-device R12
 U 1 1 5B342D6E
 P 1900 4925
@@
 $EndComp
 $Comp
-L device:R R13
+L midi-v2-circuit-rescue:R-device R13
 U 1 1 5B342D74
 P 1900 4825
@@
 	1625 4825 1750 4825
 $Comp
-L device:R R14
+L midi-v2-circuit-rescue:R-device R14
 U 1 1 5B40F987
 P 6950 5425
@@
 $EndComp
 $Comp
-L device:R R15
+L midi-v2-circuit-rescue:R-device R15
 U 1 1 5B40FFB0
 P 7125 5425
@@
 $EndComp
 $Comp
-L device:R R16
+L midi-v2-circuit-rescue:R-device R16
 U 1 1 5B41005E
 P 7300 5425
@@
 $EndComp
 $Comp
-L device:R R17
+L midi-v2-circuit-rescue:R-device R17
 U 1 1 5B410148
 P 7475 5425
